File: kicad/icarus.sch (KiCad schematic (older format))
At the start: 32 parts

Commit message: Added schematic symbols, continued schematic layout
Parts:
- added C? (x5): C_Small, symbol Device:C_Small
- added D? (x2): D_Schottky_Small, symbol Device:D_Schottky_Small
- added D? (x4): LED_Small, symbol Device:LED_Small
- added MOSFET?: PSMN4R8-100BSEJ, symbol psmn4r8-100bsej:PSMN4R8-100BSEJ
- added R?: 0.5m, symbol Device:R_Small
- added R? (x8): R_Small, symbol Device:R_Small
- added R?: 470k, symbol Device:R_Small
- added U?: LT1787HVIMS8PBF, symbol lt1787hvims8pbf:LT1787HVIMS8PBF
Connections:
- net +24V: now also C?.1, D?.1 (K), R?.1, R?.2, U?.7 (VS+)
- net +3V3: now also U?.20 (VREF+), D?.2 (A), D?.2 (A)
- net +VSW: now also C?.1, D?.1 (K), MOSFET?.3 (S), R?.2
- net EN: now also R?.1, R?.2
- net GATE: now also R?.1
- net GND: now also C?.2, C?.2, C?.2, C?.2, D?.2 (A), D?.2 (A), R?.2, R?.2, R?.2, R?.2, R?.2, U?.4 (VEE)
- net NRST: now also C?.1
- net PG: now also R?.1
- net VSENSE_LOW: now reaches U?.9 (SENSE)
- net VSENSE_LOW: now also MOSFET?.2 (D), R?.1, U?.2 (VS-)
- new net: MOSFET?.1 (G), R?.2
- new net: D?.1 (K), R?.1 (x4)
- new net: C?.2, U?.1 (FIL-)
- new net: R?.1, U?.6 (VBIAS)
- new net: C?.1, U?.8 (FIL+)
- new net: C?.1, R?.2
- new net LED1: D?.2 (A)
- new net LED2: D?.2 (A)
Other:
- note added: "CAN Bus"
- note added: "Interfaces"
- note added: "Logic Voltage Regulator"
- note added: "Microcontroller"
- note added: "Power Switching"
- note added: "Programming and Debug Hardware"
- note added: "Sensing"
- moved on the sheet: C?, H?, L?, R?, U?, U?A, U?B

Commit message: Added voltage sensing
Parts:
- removed D?: D_Schottky_Small, symbol Device:D_Schottky_Small
- added C?: 0.1uF, symbol Device:C_Small
- added C? (x3): C_Small, symbol Device:C_Small
- added D?: D_Schottky_Small, symbol Device:D_Schottky_Small
- added MOSFET? (x2): PSMN4R8-100BSEJ, symbol psmn4r8-100bsej:PSMN4R8-100BSEJ
- added R? (x4): R_Small, symbol Device:R_Small
- added U?: XT30, symbol xt30:XT30
- added U?: STLM20DD9FUDFN-4L_STM-L, symbol stlm20dd9fudfn-4l_stm-l:STLM20DD9FUDFN-4L_STM-L
- added U?: FSV10150VTO277-3L_ONS-L, symbol fsv10150vto277-3l_ons-l:FSV10150VTO277-3L_ONS-L
Connections:
- net +24V: now also U?.2 (EN/UVLO), D?.1 (K), R?.1, U?.+
- net +3V3: now also C?.1, C?.1, U?.4 (VCC)
- net +5V: now also D?.2 (A)
- net +VSW: now also MOSFET?.3 (S), MOSFET?.3 (S), R?.1, U?.3 (CATHODE)
- net CAN_SHDN: now also U?.45 (PB7)
- net GND: now also C?.2, C?.2, C?.2, C?.2, R?.2, R?.2, U?.-, U?.1 (ANODE), U?.2 (ANODE_2), U?.3 (GND)
- net VSENSE_LOW: now also MOSFET?.2 (D), MOSFET?.2 (D)
- net MOSFET_TEMP: now reaches U?.8 (PA0)
- net MOSFET_TEMP: now also U?.1 (VOUT)
- net I_SENSE_BIAS: now reaches U?.9 (PA1)
- net I_SENSE_BIAS: now also R?.1, U?.6 (VBIAS)
- net at MOSFET?.1 (G), R?.2: now also MOSFET?.1 (G), MOSFET?.1 (G)
- net I_SENSE: now reaches U?.5 (VOUT)
- new net 24V_SENSE: C?.1, R?.1, R?.2
- new net VSW_SENSE: C?.1, R?.1, R?.2
Other:
- note added: "Current Sensing"
- note added: "Temperature Sensing"
- moved on the sheet: C?, D?, H?, J?, L?, R?, U?

Commit message: Added mosfets to power driver enable, added parts values
Parts:
- removed MOSFET? (x3): PSMN4R8-100BSEJ, symbol psmn4r8-100bsej:PSMN4R8-100BSEJ
- added M1, M2, M3, M4: TPH, symbol N_Channel_MOSFET:TPH
- added R3: 47k, 1%, symbol Device:R_Small
- added R4, R9: 100k, symbol Device:R_Small
- added U5: P-CHANNEL_FET_SOT-23-3, symbol p-channel_fet_sot-23-3:P-CHANNEL_FET_SOT-23-3
- C1, C10, C11, C12, C14, C15, C5, C9: renamed from C?; value C_Small -> 0.1uF
- C13: renamed from C?; value C_Small -> 10nF
- C17, C18: renamed from C?; value C_Small -> 0.01uF
- C2, C4, C7: renamed from C?; value C_Small -> 1uF, 100V
- C3: renamed from C?; value C_Small -> 10uF
- C6: renamed from C?; value C_Small -> 0.1uF, 100V
- C8: renamed from C?; value C_Small -> 1uF
- L1: renamed from L?; value L_Small -> 33uH
- R10: renamed from R?; value R_Small -> 140k, 1%
- R11, R12, R5, R6: renamed from R?; value R_Small -> 220
- R13: renamed from R?; value R_Small -> 47k, 1%
- R14: renamed from R?; value R_Small -> 6.8k, 1%
- R16, R17: renamed from R?; value R_Small -> 3M, 1%
- R18, R19: renamed from R?; value R_Small -> 200k, 1%
- R7: renamed from R?; value R_Small -> 10
- R8: renamed from R?; value R_Small -> 499k, 1%
- gave numbers to parts that had none: 33
Connections:
- net +24V: now also R3.2, U5.P$3 (DRAIN); no longer R8.1
- net +VSW: now also M1.1 (S), M1.2 (S), M1.3 (S), M2.1 (S), M2.2 (S), M2.3 (S), M4.1 (S), M4.2 (S), M4.3 (S)
- net GND: now also M3.1 (S), M3.2 (S), M3.3 (S), R9.2
- net VSENSE_LOW: now also M1.5 (D), M1.6 (D), M1.7 (D), M1.8 (D), M1.EP (D), M2.5 (D), M2.6 (D), M2.7 (D), M2.8 (D), M2.EP (D), M4.5 (D), M4.6 (D), M4.7 (D), M4.8 (D), M4.EP (D)
- net at R7.2: now also M1.4 (G), M2.4 (G), M4.4 (G)
- new net: R8.1, U5.P$2 (SOURCE)
- new net: R3.1, R4.2, U5.P$1 (GATE)
- new net: M3.5 (D), M3.6 (D), M3.7 (D), M3.8 (D), M3.EP (D), R4.1
- new net TPS_ENABLE: M3.4 (G), R9.1
Other:
- moved on the sheet: C13, C6, C7, D2, D3, D4, D5, D6, H1, H2, H3, H4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

Commit message: Updated schematic and CubeMX pinouts
Parts:
- added C13: 10uF, symbol Device:C_Small
- added D7, D8: LED_Small, symbol Device:LED_Small
- added R13, R14: 220, symbol Device:R_Small
- renumbered C13 to C14, C14 to C15, C15 to C16, C16 to C17, C17 to C18, C18 to C19, R13 to R15, R14 to R16, R15 to R17, R16 to R18, R17 to R19, R18 to R20, R19 to R21, R7 to R4, R4 to R5, R5 to R6, R6 to R7, U8 to U10, U10 to U11, U11 to U12, U12 to U13, U13 to U14, U14 to U15, U15 to U16, U5 to U4, U4 to U5, U7 to U6, 1 to U7, U6 to U8
Connections:
- net +3V3: now also D5.2 (A), D6.2 (A), C13.1, D7.2 (A), D8.2 (A)
- net 24V_SENSE: now also U2.18 (PB1)
- net GND: now also U2.49 (EPAD); no longer C10.2, C11.2, C12.2, C8.2, C9.2, R11.2, R12.2
- net I_SENSE: now also U2.10 (PA2)
- net LED1: now also R11.2, U2.11 (PA3); no longer D5.2 (A)
- net LED2: now also R12.2, U2.13 (PA5); no longer D6.2 (A)
- net TPS_ENABLE: now also U2.44 (PB6)
- net VSW_SENSE: now also U2.19 (PB2)
- net LED3: now reaches U2.15 (PA7)
- net LED3: now also R13.2
- net LED4: now reaches U2.17 (PB0)
- net LED4: now also R14.2
- new net: C10.2, C11.2, C12.2, C13.2, C8.2, C9.2
- new net: D7.1 (K), R13.1
- new net: D8.1 (K), R14.1
- no-connect marks 4 -> 27
Other:
- note added: "XT30s"
- note added: "XT90"
- moved on the sheet: R2, R4
