File: kicad/icarus.sch (KiCad schematic (older format))
At the start: 78 parts, among them J1 CAN Bus, J2 CAN Bus, J3 SWD Programming, J4 USB_B_Micro, M1 PSMN4R8-100BSEJ, M2 PSMN4R8-100BSEJ, M3 BSS123, M4 PSMN4R8-100BSEJ, U1 MAX15062A, U10 XT30, U11 XT30, U12 XT30, U13 XT30, U14 LT1787HVIMS8PBF, U15 USBLC6-2SC6, U16 STLM20DD9FUDFN-4L_STM-L, U2 STM32G474CEU6, U3 TCAN334G, U4 ZXMP10A13FTA, U5 XT90, U6 FSV10150VTO277-3L_ONS-L, U7 XT30, U8 XT30, U9 TPS2490DGSR

Commit message: Added and assigned footprints, generated netlist
Parts:
- C1, C10, C11, C12, C13, C14, C15, C16, C17, C18, C19, C3, C5, C6, C8, C9: footprint (none) -> Capacitor_SMD:C_0402_1005Metric
- C2, C4, C7: footprint (none) -> Capacitor_SMD:C_0805_2012Metric
- D1: footprint (none) -> Diode_SMD:D_SOD-523
- D2: footprint (none) -> icarus_kicad_lib:SMBJ51CA-E3-52214AB
- D3: renamed from D?; footprint (none) -> icarus_kicad_lib:SMBJ51CA-E3-52214AB
- D4: renamed from D3; footprint (none) -> LED_SMD:LED_0603_1608Metric
- D5: renamed from D4; footprint (none) -> LED_SMD:LED_0603_1608Metric
- D6: renamed from D5; footprint (none) -> LED_SMD:LED_0603_1608Metric
- D7: renamed from D6; footprint (none) -> LED_SMD:LED_0603_1608Metric
- D8: renamed from D7; footprint (none) -> LED_SMD:LED_0603_1608Metric
- D9: renamed from D8; footprint (none) -> LED_SMD:LED_0603_1608Metric
- H1, H2, H3, H4: footprint (none) -> MountingHole:MountingHole_2.7mm_M2.5_DIN965_Pad
- J1, J2: footprint (none) -> Connector_JST:JST_PH_S3B-PH-SM4-TB_1x03-1MP_P2.00mm_Horizontal
- J3: footprint (none) -> Connector_JST:JST_PH_S6B-PH-K_1x06_P2.00mm_Horizontal
- J4: footprint (none) -> Connector_USB:USB_Micro-AB_Molex_47590-0001
- L1: footprint (none) -> Inductor_SMD:L_1210_3225Metric
- M1, M2, M4: footprint (none) -> icarus_kicad_lib:PSMN4R8-100BSEJ
- M3, U4: footprint (none) -> Package_TO_SOT_SMD:SOT-23
- R1, R10, R11, R12, R13, R14, R15, R16, R17, R2, R20, R21, R3, R4, R5, R6, R7, R8, R9: footprint (none) -> Resistor_SMD:R_0402_1005Metric
- R18, R19: footprint (none) -> Resistor_SMD:R_0603_1608Metric
- U10, U11, U12, U13, U7, U8: footprint (none) -> icarus_kicad_lib:XT30P
- U14: footprint (none) -> icarus_kicad_lib:LT1787HVIMS8PBF
- U16: footprint (none) -> icarus_kicad_lib:STLM20DD9FUDFN-4L_STM-L
- U3: footprint (none) -> icarus_kicad_lib:TCAN334G
- U5: footprint (none) -> icarus_kicad_lib:XT90PW-M
- U6: footprint (none) -> icarus_kicad_lib:FSV10150VTO277-3L_ONS-L
- U9: footprint (none) -> icarus_kicad_lib:TPS2490DGSR

Commit message: Began fixing footprint disasters:
Parts:
- removed D1: RB520S30, Diode_SMD:D_SOD-523, symbol Device:D_Schottky_Small
- removed D2, D3: SMBJ51CA-E3/52, icarus_kicad_lib:SMBJ51CA-E3-52214AB, symbol Device:D_Schottky_Small
- removed M1, M2, M4: PSMN4R8-100BSEJ, icarus_kicad_lib:PSMN4R8-100BSEJ, symbol N_Channel_MOSFET:TPH
- removed M3: BSS123, Package_TO_SOT_SMD:SOT-23, symbol N_Channel_MOSFET:TPH
- added CR1, CR2: SMBJ51CA-E3_52, icarus_kicad_lib:SMBJ51CA-E3-52, symbol SMBJ51CA-E3&slash_52:SMBJ51CA-E3_52
- added D1: RB520S30, icarus_kicad_lib:RB520S30, symbol RB520S30:RB520S30
- added MOSFET1, MOSFET2, MOSFET3: PSMN4R8-100BSEJ, icarus_kicad_lib:PSMN4R8-100BSEJ, symbol icarus-rescue:PSMN4R8-100BSEJ-psmn4r8-100bsej
- added Q1: BSS123, digikey-footprints:SOT-23-3, symbol dk_Transistors-FETs-MOSFETs-Single:BSS123
- J1, J2: footprint Connector_JST:JST_PH_S3B-PH-SM4-TB_1x03-1MP_P2.00mm_Horizontal -> Connector_JST:JST_PH_B3B-PH-SM4-TB_1x03-1MP_P2.00mm_Vertical
- J3: footprint Connector_JST:JST_PH_S6B-PH-K_1x06_P2.00mm_Horizontal -> Connector_JST:JST_PH_B6B-PH-K_1x06_P2.00mm_Vertical
- U15: footprint Package_TO_SOT_SMD:SOT-23-6 -> digikey-footprints:SOT-23-6
- U2: footprint UFQFPN-48_7X7X0P55MM -> icarus_kicad_lib:STM32G474CEU6
- U4: footprint Package_TO_SOT_SMD:SOT-23 -> digikey-footprints:SOT-23-3
Other:
- moved on the sheet: R4
Changed lines of the file:
@@
 F 0 "U2" H 2050 5912 60  0000 C CNN
 F 1 "STM32G474CEU6" H 2050 5806 60  0000 C CNN
-F 2 "UFQFPN-48_7X7X0P55MM" H 2650 5765 60  0001 C CNN
+F 2 "icarus_kicad_lib:STM32G474CEU6" H 2650 5765 60  0001 C CNN
 F 3 "" H 1250 5525 60  0000 C CNN
 	2    1250 5525
@@
 F 0 "J1" H 14055 3342 50  0000 L CNN
 F 1 "CAN Bus" H 14055 3251 50  0000 L CNN
-F 2 "Connector_JST:JST_PH_S3B-PH-SM4-TB_1x03-1MP_P2.00mm_Horizontal" H 13975 3300 50  0001 C CNN
+F 2 "Connector_JST:JST_PH_B3B-PH-SM4-TB_1x03-1MP_P2.00mm_Vertical" H 13975 3300 50  0001 C CNN
 F 3 "~" H 13975 3300 50  0001 C CNN
 	1    13975 3300
@@
 F 0 "J2" H 15230 3342 50  0000 L CNN
 F 1 "CAN Bus" H 15230 3251 50  0000 L CNN
-F 2 "Connector_JST:JST_PH_S3B-PH-SM4-TB_1x03-1MP_P2.00mm_Horizontal" H 15150 3300 50  0001 C CNN
+F 2 "Connector_JST:JST_PH_B3B-PH-SM4-TB_1x03-1MP_P2.00mm_Vertical" H 15150 3300 50  0001 C CNN
 F 3 "~" H 15150 3300 50  0001 C CNN
 	1    15150 3300
@@
 F 0 "U15" H 4950 8575 50  0000 C CNN
 F 1 "USBLC6-2SC6" H 5175 8500 50  0000 C CNN
-F 2 "Package_TO_SOT_SMD:SOT-23-6" H 4800 8425 50  0001 C CNN
+F 2 "digikey-footprints:SOT-23-6" H 4800 8425 50  0001 C CNN
 F 3 "https://www.st.com/resource/en/datasheet/usblc6-2.pdf" H 5000 9275 50  0001 C CNN
 	1    4800 8925
@@
 F 0 "J3" H 1480 8892 50  0000 L CNN
 F 1 "SWD Programming" H 1480 8801 50  0000 L CNN
-F 2 "Connector_JST:JST_PH_S6B-PH-K_1x06_P2.00mm_Horizontal" H 1400 8900 50  0001 C CNN
+F 2 "Connector_JST:JST_PH_B6B-PH-K_1x06_P2.00mm_Vertical" H 1400 8900 50  0001 C CNN
 F 3 "~" H 1400 8900 50  0001 C CNN
 	1    1400 8900
@@
 F 0 "U2" H 2650 1912 60  0000 C CNN
 F 1 "STM32G474CEU6" H 2650 1806 60  0000 C CNN
-F 2 "UFQFPN-48_7X7X0P55MM" H 2650 1765 60  0001 C CNN
+F 2 "icarus_kicad_lib:STM32G474CEU6" H 2650 1765 60  0001 C CNN
 F 3 "" H 1250 1525 60  0000 C CNN
 	1    1250 1525
@@
 	7625 1300 8525 1300
 $Comp
-L Device:D_Schottky_Small D1
-U 1 1 60993B27
-P 7625 1200
-F 0 "D1" V 7671 1130 50  0000 R CNN
-F 1 "RB520S30" V 7580 1130 50  0000 R CNN
-F 2 "Diode_SMD:D_SOD-523" V 7625 1200 50  0001 C CNN
-F 3 "~" V 7625 1200 50  0001 C CNN
-	1    7625 1200
-	0    -1   -1   0
-$EndComp
-$Comp
 L power:+5V #PWR0141
 U 1 1 6098DBDE
@@
 $EndComp
 $Comp
-L Device:D_Schottky_Small D2
-U 1 1 60596EE2
-P 7525 3625
-F 0 "D2" V 7525 3700 50  0000 L CNN
-F 1 "SMBJ51CA-E3/52" V 7350 3300 50  0000 L CNN
-F 2 "icarus_kicad_lib:SMBJ51CA-E3-52214AB" V 7525 3625 50  0001 C CNN
-F 3 "~" V 7525 3625 50  0001 C CNN
-	1    7525 3625
-	0    1    1    0
-$EndComp
-$Comp
 L power:+24V #PWR0143
 U 1 1 60599BA2
@@
 L power:GND #PWR0145
 U 1 1 605E1459
-P 7650 3725
-F 0 "#PWR0145" H 7650 3475 50  0001 C CNN
-F 1 "GND" H 7655 3552 50  0000 C CNN
-F 2 "" H 7650 3725 50  0001 C CNN
-F 3 "" H 7650 3725 50  0001 C CNN
-	1    7650 3725
+P 7575 3925
+F 0 "#PWR0145" H 7575 3675 50  0001 C CNN
+F 1 "GND" H 7580 3752 50  0000 C CNN
+F 2 "" H 7575 3925 50  0001 C CNN
+F 3 "" H 7575 3925 50  0001 C CNN
+	1    7575 3925
 	1    0    0    -1
 $EndComp
 Wire Wire Line
 	7000 3525 7200 3525
-Wire Wire Line
-	7200 3525 7525 3525
 Wire Wire Line
 	8625 3525 8700 3525
@@
 Wire Wire Line
 	9650 4150 9650 4775
-Text GLabel 10150 4350 2    50   Input ~ 0
+Text GLabel 10150 4450 2    50   Input ~ 0
 GATE
 $Comp
 L Device:R_Small R4
 U 1 1 605F126E
-P 9925 4350
-F 0 "R4" V 9729 4350 50  0000 C CNN
-F 1 "10" V 9820 4350 50  0000 C CNN
-F 2 "Resistor_SMD:R_0402_1005Metric" H 9925 4350 50  0001 C CNN
-F 3 "~" H 9925 4350 50  0001 C CNN
-	1    9925 4350
+P 9925 4450
+F 0 "R4" V 9729 4450 50  0000 C CNN
+F 1 "10" V 9820 4450 50  0000 C CNN
+F 2 "Resistor_SMD:R_0402_1005Metric" H 9925 4450 50  0001 C CNN
+F 3 "~" H 9925 4450 50  0001 C CNN
+	1    9925 4450
 	0    1    1    0
 $EndComp
@@
 F 0 "U4" H 8553 4250 40  0000 L CNN
 F 1 "ZXMP10A13FTA" H 8553 4212 40  0001 L CNN
-F 2 "Package_TO_SOT_SMD:SOT-23" H 8375 4250 50  0001 C CNN
+F 2 "digikey-footprints:SOT-23-3" H 8375 4250 50  0001 C CNN
 F 3 "" H 8375 4250 50  0001 C CNN
 	1    8375 4250
@@
 Wire Wire Line
 	8175 3950 8475 3950
-$Comp
-L N_Channel_MOSFET:TPH M1
-U 1 1 60D0211C
-P 9375 3625
-F 0 "M1" V 9625 3625 59  0000 C CNN
-F 1 "PSMN4R8-100BSEJ" H 9573 3573 59  0001 L CNN
-F 2 "icarus_kicad_lib:PSMN4R8-100BSEJ" H 9375 3625 50  0001 C CNN
-F 3 "" H 9375 3625 50  0001 C CNN
-	1    9375 3625
-	0    -1   -1   0
-$EndComp
-$Comp
-L N_Channel_MOSFET:TPH M2
-U 1 1 60D185B1
-P 9375 4250
-F 0 "M2" V 9625 4250 59  0000 C CNN
-F 1 "PSMN4R8-100BSEJ" H 9573 4198 59  0001 L CNN
-F 2 "icarus_kicad_lib:PSMN4R8-100BSEJ" H 9375 4250 50  0001 C CNN
-F 3 "" H 9375 4250 50  0001 C CNN
-	1    9375 4250
-	0    -1   -1   0
-$EndComp
-$Comp
-L N_Channel_MOSFET:TPH M4
-U 1 1 60D196A4
-P 9375 4875
-F 0 "M4" V 9625 4875 59  0000 C CNN
-F 1 "PSMN4R8-100BSEJ" H 9573 4823 59  0001 L CNN
-F 2 "icarus_kicad_lib:PSMN4R8-100BSEJ" H 9375 4875 50  0001 C CNN
-F 3 "" H 9375 4875 50  0001 C CNN
-	1    9375 4875
-	0    -1   -1   0
-$EndComp
-$Comp
-L N_Channel_MOSFET:TPH M3
-U 1 1 60D33111
-P 7800 4725
-F 0 "M3" H 7998 4725 59  0000 L CNN
-F 1 "BSS123" H 7998 4673 59  0001 L CNN
-F 2 "Package_TO_SOT_SMD:SOT-23" H 7800 4725 50  0001 C CNN
-F 3 "" H 7800 4725 50  0001 C CNN
-	1    7800 4725
-	1    0    0    -1
-$EndComp
-Wire Wire Line
-	7700 4825 7400 4825
 Wire Wire Line
 	7400 4825 7400 4850
 Wire Wire Line
 	7275 4825 7400 4825
-Connection ~ 7400 4825
 Wire Wire Line
 	8175 3525 8175 3950
@@
 	-1   0    0    1
 $EndComp
-Wire Wire Line
-	9475 4975 9750 4975
-Wire Wire Line
-	9475 3725 9750 3725
 Connection ~ 10450 3525
 Wire Wire Line
@@
 	9650 3525 10450 3525
 Wire Wire Line
-	9750 3725 9750 4350
-Wire Wire Line
-	9475 4350 9750 4350
-Connection ~ 9750 4350
-Wire Wire Line
-	9750 4350 9750 4975
-Wire Wire Line
-	9825 4350 9750 4350
-Wire Wire Line
-	10025 4350 10150 4350
+	10025 4450 10150 4450
 NoConn ~ 1250 1925
 NoConn ~ 1250 2125
@@
 NoConn ~ 4050 1625
 NoConn ~ 4050 1525
-Connection ~ 7525 3525
-Wire Wire Line
-	7525 3525 7775 3525
-$Comp
-L Device:D_Schottky_Small D3
-U 1 1 60754BF1
-P 7775 3625
-F 0 "D3" V 7775 3700 50  0000 L CNN
-F 1 "SMBJ51CA-E3/52" V 7600 3300 50  0000 L CNN
-F 2 "icarus_kicad_lib:SMBJ51CA-E3-52214AB" V 7775 3625 50  0001 C CNN
-F 3 "~" V 7775 3625 50  0001 C CNN
-	1    7775 3625
+$Comp
+L icarus-rescue:PSMN4R8-100BSEJ-psmn4r8-100bsej MOSFET1
+U 1 1 608852C7
+P 9375 3825
+F 0 "MOSFET1" V 9877 3825 85  0000 C CNN
+F 1 "PSMN4R8-100BSEJ" V 9877 3825 85  0001 C CNN
+F 2 "icarus_kicad_lib:PSMN4R8-100BSEJ" H 9375 3825 50  0001 C CNN
+F 3 "" H 9375 3825 50  0001 C CNN
+	1    9375 3825
+	0    -1   -1   0
+$EndComp
+$Comp
+L icarus-rescue:PSMN4R8-100BSEJ-psmn4r8-100bsej MOSFET2
+U 1 1 6088724D
+P 9375 4450
+F 0 "MOSFET2" V 9877 4450 85  0000 C CNN
+F 1 "PSMN4R8-100BSEJ" V 9877 4450 85  0001 C CNN
+F 2 "icarus_kicad_lib:PSMN4R8-100BSEJ" H 9375 4450 50  0001 C CNN
+F 3 "" H 9375 4450 50  0001 C CNN
+	1    9375 4450
+	0    -1   -1   0
+$EndComp
+$Comp
+L icarus-rescue:PSMN4R8-100BSEJ-psmn4r8-100bsej MOSFET3
+U 1 1 60888AB1
+P 9375 5075
+F 0 "MOSFET3" V 9877 5075 85  0000 C CNN
+F 1 "PSMN4R8-100BSEJ" V 9877 5075 85  0001 C CNN
+F 2 "icarus_kicad_lib:PSMN4R8-100BSEJ" H 9375 5075 50  0001 C CNN
+F 3 "" H 9375 5075 50  0001 C CNN
+	1    9375 5075
+	0    -1   -1   0
+$EndComp
+Wire Wire Line
+	9375 3825 9750 3825
+Wire Wire Line
+	9375 4450 9750 4450
+Connection ~ 9750 4450
+Wire Wire Line
+	9750 3825 9750 4450
+Wire Wire Line
+	9825 4450 9750 4450
+Wire Wire Line
+	9375 5075 9750 5075
+Wire Wire Line
+	9750 4450 9750 5075
+Wire Wire Line
+	7200 3525 7475 3525
+$Comp
+L SMBJ51CA-E3&slash_52:SMBJ51CA-E3_52 CR1
+U 1 1 608E4AFE
+P 7475 3925
+F 0 "CR1" V 7728 3821 60  0000 R CNN
+F 1 "SMBJ51CA-E3_52" V 7622 3821 60  0000 R CNN
+F 2 "icarus_kicad_lib:SMBJ51CA-E3-52" H 7675 3565 60  0001 C CNN
+F 3 "" H 7475 3925 60  0000 C CNN
+	1    7475 3925
+	0    -1   -1   0
+$EndComp
+Connection ~ 7475 3525
+$Comp
+L SMBJ51CA-E3&slash_52:SMBJ51CA-E3_52 CR2
+U 1 1 608F0D36
+P 7675 3925
+F 0 "CR2" V 7928 3821 60  0000 R CNN
+F 1 "SMBJ51CA-E3_52" V 7822 3821 60  0000 R CNN
+F 2 "icarus_kicad_lib:SMBJ51CA-E3-52" H 7875 3565 60  0001 C CNN
+F 3 "" H 7675 3925 60  0000 C CNN
+	1    7675 3925
+	0    -1   -1   0
+$EndComp
+Connection ~ 7675 3525
+Wire Wire Line
+	7675 3525 8175 3525
+Wire Wire Line
+	7475 3925 7575 3925
+Wire Wire Line
+	7475 3525 7675 3525
+Connection ~ 7575 3925
+Wire Wire Line
+	7575 3925 7675 3925
+$Comp
+L dk_Transistors-FETs-MOSFETs-Single:BSS123 Q1
+U 1 1 60925E78
+P 7900 4725
+F 0 "Q1" H 8008 4778 60  0000 L CNN
+F 1 "BSS123" H 8008 4672 60  0000 L CNN
+F 2 "digikey-footprints:SOT-23-3" H 8100 4925 60  0001 L CNN
+F 3 "https://www.onsemi.com/pub/Collateral/BSS123-D.PDF" H 8100 5025 60  0001 L CNN
+F 4 "BSS123NCT-ND" H 8100 5125 60  0001 L CNN "Digi-Key_PN"
+F 5 "BSS123" H 8100 5225 60  0001 L CNN "MPN"
+F 6 "Discrete Semiconductor Products" H 8100 5325 60  0001 L CNN "Category"
+F 7 "Transistors - FETs, MOSFETs - Single" H 8100 5425 60  0001 L CNN "Family"
+F 8 "https://www.onsemi.com/pub/Collateral/BSS123-D.PDF" H 8100 5525 60  0001 L CNN "DK_Datasheet_Link"
+F 9 "/product-detail/en/on-semiconductor/BSS123/BSS123NCT-ND/244665" H 8100 5625 60  0001 L CNN "DK_Detail_Page"
+F 10 "MOSFET N-CH 100V 170MA SOT-23" H 8100 5725 60  0001 L CNN "Description"
+F 11 "ON Semiconductor" H 8100 5825 60  0001 L CNN "Manufacturer"
+F 12 "Active" H 8100 5925 60  0001 L CNN "Status"
+	1    7900 4725
+	1    0    0    -1
+$EndComp
+Wire Wire Line
+	7600 4825 7400 4825
+Connection ~ 7400 4825
+$Comp
+L RB520S30:RB520S30 D1
+U 1 1 6094C802
+P 7625 1200
+F 0 "D1" V 7579 1280 50  0000 L CNN
+F 1 "RB520S30" V 7670 1280 50  0000 L CNN
+F 2 "icarus_kicad_lib:RB520S30" H 7625 1200 50  0001 L BNN
+F 3 "" H 7625 1200 50  0001 L BNN
+	1    7625 1200
 	0    1    1    0
 $EndComp
-Connection ~ 7775 3525
-Wire Wire Line
-	7775 3525 8175 3525
-Wire Wire Line
-	7525 3725 7650 3725
-Connection ~ 7650 3725
-Wire Wire Line
-	7650 3725 7775 3725
 $EndSCHEMATC
