File: kicad/_autosave-icarus.sch (KiCad schematic (older format))
At the start: 78 parts, among them J1 CAN Bus, J2 CAN Bus, J3 SWD Programming, J4 USB_B_Micro, M1 PSMN4R8-100BSEJ, M2 PSMN4R8-100BSEJ, M3 BSS123, M4 PSMN4R8-100BSEJ, U1 MAX15062A, U10 XT30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

Commit message: Added initial BOM
Parts:
- gave numbers to parts that had none: 1
- renumbered D3 to D4, D4 to D5, D5 to D6, D6 to D7, D7 to D8, D8 to D9
Changed lines of the file:
@@
 $EndComp
 $Comp
-L Device:LED_Small D4
+L Device:LED_Small D5
 U 1 1 607A30EE
 P 5500 4250
-F 0 "D4" V 5546 4180 50  0000 R CNN
+F 0 "D5" V 5546 4180 50  0000 R CNN
 F 1 "Green" V 5455 4180 50  0000 R CNN
 F 2 "" V 5500 4250 50  0001 C CNN
@@
 $EndComp
 $Comp
-L Device:LED_Small D5
+L Device:LED_Small D6
 U 1 1 607B09D4
 P 4925 5175
-F 0 "D5" V 4971 5105 50  0000 R CNN
+F 0 "D6" V 4971 5105 50  0000 R CNN
 F 1 "Blue" V 4880 5105 50  0000 R CNN
 F 2 "" V 4925 5175 50  0001 C CNN
@@
 $EndComp
 $Comp
-L Device:LED_Small D3
+L Device:LED_Small D4
 U 1 1 607D3F96
 P 4925 4250
-F 0 "D3" V 4971 4180 50  0000 R CNN
+F 0 "D4" V 4971 4180 50  0000 R CNN
 F 1 "Green" V 4880 4180 50  0000 R CNN
 F 2 "" V 4925 4250 50  0001 C CNN
@@
 $EndComp
 $Comp
-L Device:LED_Small D6
+L Device:LED_Small D7
 U 1 1 607DF041
 P 5500 5175
-F 0 "D6" V 5546 5105 50  0000 R CNN
+F 0 "D7" V 5546 5105 50  0000 R CNN
 F 1 "Blue" V 5455 5105 50  0000 R CNN
 F 2 "" V 5500 5175 50  0001 C CNN
@@
 Connection ~ 3225 6750
 $Comp
-L Device:LED_Small D7
+L Device:LED_Small D8
 U 1 1 604C7C67
 P 4925 6150
-F 0 "D7" V 4971 6080 50  0000 R CNN
+F 0 "D8" V 4971 6080 50  0000 R CNN
 F 1 "Blue" V 4880 6080 50  0000 R CNN
 F 2 "" V 4925 6150 50  0001 C CNN
@@
 LED3
 $Comp
-L Device:LED_Small D8
+L Device:LED_Small D9
 U 1 1 604C7C7B
 P 5500 6150
-F 0 "D8" V 5546 6080 50  0000 R CNN
+F 0 "D9" V 5546 6080 50  0000 R CNN
 F 1 "Blue" V 5455 6080 50  0000 R CNN
 F 2 "" V 5500 6150 50  0001 C CNN
@@
 	7525 3525 7775 3525
 $Comp
-L Device:D_Schottky_Small D?
+L Device:D_Schottky_Small D3
 U 1 1 60754BF1
 P 7775 3625
-F 0 "D?" V 7775 3700 50  0000 L CNN
+F 0 "D3" V 7775 3700 50  0000 L CNN
 F 1 "SMBJ51CA-E3/52" V 7600 3300 50  0000 L CNN
 F 2 "" V 7775 3625 50  0001 C CNN
